File: 2065-Z80-programmer.sch (KiCad schematic (older format))
At the start: 31 parts, among them J1 Conn_01x05, J2 Conn_02x20_Counter_Clockwise, J3 Conn_01x02, J4 Conn_02x20_Odd_Even, Q1 2N7000, Q2 2N7000, Q3 PN2222, U1 MCP23017-E_SP, U2 MCP23017-E_SP

Commit message: Change Digikey part numbers on 1x5 header
Parts:
- J1: Digi-Key_PN S1211EC-05-ND -> S1011EC-05-ND; MPN (none) -> PRPC005SAAN-RC; Manufacturer (none) -> Sullins Connector Solutions
Changed lines of the file:
@@
 F 3 "https://media.digikey.com/PDF/Data%20Sheets/Sullins%20PDFs/xRxCzzzSxxN-RC_ST_11635-B.pdf" H 1050 1600 50  0001 C CNN
 F 4 "Generic connector, single row, 01x05" H 1050 1600 50  0001 C CNN "Description"
-F 5 "S1211EC-05-ND" H 1050 1600 50  0001 C CNN "Digi-Key_PN"
+F 5 "S1011EC-05-ND" H 1050 1600 50  0001 C CNN "Digi-Key_PN"
+F 6 "PRPC005SAAN-RC" H 1050 1600 50  0001 C CNN "MPN"
+F 7 "Sullins Connector Solutions" H 1050 1600 50  0001 C CNN "Manufacturer"
 	1    1050 1600
 	-1   0    0    1
